Commit message: Update to include manipulator

File: quad_description/urdf/kit_c.urdf (robot description, URDF)
Before this commit: robot quad, 6 links, 5 joints
Links:
- added link left_finger, mass 0.1; collision box size=0.025 0.075 0.025; visual box size=0.025 0.075 0.025
- added link left_finger_tip, mass 0.1; collision box size=0.025 0.05 0.025; visual box size=0.025 0.05 0.025
- added link palm, mass 0.5; collision box size=0.025 0.05 0.025; visual box size=0.025 0.05 0.025
- added link right_finger, mass 0.1; collision box size=0.025 0.075 0.025; visual box size=0.025 0.075 0.025
- added link right_finger_tip, mass 0.1; collision box size=0.025 0.05 0.025; visual box size=0.025 0.05 0.025
- added link riser, mass 10; collision box size=0.025 0.025 0.25; visual box size=0.025 0.025 0.25
Joints:
- added joint base1_joint: type fixed, parent base_link, child riser, origin xyz=0 0 -0.1302 rpy=0 0 0
- added joint left_finger_tip: type revolute, parent left_finger, child left_finger_tip, origin xyz=0 0.025 0 rpy=0 0 0, axis 0 0 1, limit lower=-0.4 upper=0.4 effort=2.5 velocity=1.0
- added joint palm_left_finger: type revolute, parent palm, child left_finger, origin xyz=0 -0.025 0 rpy=0 0 0, axis 0 0 1, limit lower=-0.4 upper=0.4 effort=2.5 velocity=1.0
- added joint palm_right_finger: type revolute, parent palm, child right_finger, origin xyz=0 0.025 0 rpy=0 0 0, axis 0 0 1, limit lower=-0.4 upper=0.4 effort=2.5 velocity=1.0
- added joint palm_riser: type prismatic, parent riser, child palm, axis 0 0 1, limit lower=0 upper=0.9 effort=2.5 velocity=1.0
- added joint right_finger_tip: type revolute, parent right_finger, child right_finger_tip, origin xyz=0 0.025 0 rpy=0 0 0, axis 0 0 1, limit lower=-0.4 upper=0.4 effort=2.5 velocity=1.0

Commit message: urdf update

File: quad_description/urdf/kit_c.urdf (robot description, URDF)
Before this commit: robot quad, 12 links, 11 joints
Links:
- link palm: mass 0.5 -> 0.1
- link riser: mass 10 -> 0.2
Joints:
- joint base1_joint: origin xyz=0 0 -0.1302 rpy=0 0 0 -> xyz=0.025 0 -0.25 rpy=0 0 0
- joint left_finger_tip: limit lower=-0.4 upper=0.4 effort=2.5 velocity=1.0 -> lower=-0.1 upper=0.1 effort=2.5 velocity=1.0
- joint palm_left_finger: limit lower=-0.4 upper=0.4 effort=2.5 velocity=1.0 -> lower=-0.2 upper=0.2 effort=2.5 velocity=1.0
- joint palm_right_finger: limit lower=-0.4 upper=0.4 effort=2.5 velocity=1.0 -> lower=-0.2 upper=0.2 effort=2.5 velocity=1.0
- joint right_finger_tip: limit lower=-0.4 upper=0.4 effort=2.5 velocity=1.0 -> lower=-0.1 upper=0.1 effort=2.5 velocity=1.0

Commit message: palm_riser joint origin update

File: quad_description/urdf/kit_c.urdf (robot description, URDF)
Before this commit: robot quad, 12 links, 11 joints
Joints:
- joint palm_riser: origin (none) -> xyz=0 0.025 0 rpy=0 0 0

File: quad_description/urdf/my_gripper.xacro (robot description, xacro)
@@ -162,4 +162,5 @@
       <axis xyz="0 0 1"/>
       <limit lower="0" upper="0.9" effort="2.5" velocity="1.0"/>
+      <origin rpy="0 0 0" xyz="0 0.025 0"/>
       <parent link="riser"/>
       <child link="palm"/>

Commit message: added seperate controllers

File: quad_description/urdf/kit_c.urdf (robot description, URDF)
Before this commit: robot quad, 12 links, 11 joints
Joints:
- joint palm_riser: limit lower=0 upper=0.9 effort=2.5 velocity=1.0 -> lower=0 upper=0.1 effort=2.5 velocity=1.0; origin xyz=0 0.025 0 rpy=0 0 0 -> xyz=0 0 0 rpy=0 0 0

File: quad_description/urdf/my_gripper.xacro (robot description, xacro)
@@ -161,6 +161,6 @@
     <joint name="palm_riser" type="prismatic">
       <axis xyz="0 0 1"/>
-      <limit lower="0" upper="0.9" effort="2.5" velocity="1.0"/>
-      <origin rpy="0 0 0" xyz="0 0.025 0"/>
+      <limit lower="0" upper="0.1" effort="2.5" velocity="1.0"/>
+      <origin rpy="0 0 0" xyz="0 0 0"/>
       <parent link="riser"/>
       <child link="palm"/>
@@ -170,8 +170,8 @@
       <type>transmission_interface/SimpleTransmission</type>
       <joint name="palm_left_finger">
-        <hardwareInterface>EffortJointInterface</hardwareInterface>
+        <hardwareInterface>PositionJointInterface</hardwareInterface>
       </joint>
       <actuator name="motor1">
-        <hardwareInterface>EffortJointInterface</hardwareInterface>
+        <hardwareInterface>PositionJointInterface</hardwareInterface>
         <mechanicalReduction>1</mechanicalReduction>
       </actuator>
@@ -180,8 +180,8 @@
       <type>transmission_interface/SimpleTransmission</type>
       <joint name="left_finger_tip">
-        <hardwareInterface>EffortJointInterface</hardwareInterface>
+        <hardwareInterface>PositionJointInterface</hardwareInterface>
       </joint>
       <actuator name="motor2">
-        <hardwareInterface>EffortJointInterface</hardwareInterface>
+        <hardwareInterface>PositionJointInterface</hardwareInterface>
         <mechanicalReduction>1</mechanicalReduction>
       </actuator>
@@ -190,8 +190,8 @@
       <type>transmission_interface/SimpleTransmission</type>
       <joint name="palm_right_finger">
-        <hardwareInterface>EffortJointInterface</hardwareInterface>
+        <hardwareInterface>PositionJointInterface</hardwareInterface>
       </joint>
       <actuator name="motor3">
-        <hardwareInterface>EffortJointInterface</hardwareInterface>
+        <hardwareInterface>PositionJointInterface</hardwareInterface>
         <mechanicalReduction>1</mechanicalReduction>
       </actuator>
@@ -200,8 +200,8 @@
       <type>transmission_interface/SimpleTransmission</type>
       <joint name="right_finger_tip">
-        <hardwareInterface>EffortJointInterface</hardwareInterface>
+        <hardwareInterface>PositionJointInterface</hardwareInterface>
       </joint>
       <actuator name="motor4">
-        <hardwareInterface>EffortJointInterface</hardwareInterface>
+        <hardwareInterface>PositionJointInterface</hardwareInterface>
         <mechanicalReduction>1</mechanicalReduction>
       </actuator>
@@ -210,8 +210,8 @@
       <type>transmission_interface/SimpleTransmission</type>
       <joint name="palm_riser">
-        <hardwareInterface>EffortJointInterface</hardwareInterface>
+        <hardwareInterface>PositionJointInterface</hardwareInterface>
       </joint>
       <actuator name="motor5">
-        <hardwareInterface>EffortJointInterface</hardwareInterface>
+        <hardwareInterface>PositionJointInterface</hardwareInterface>
         <mechanicalReduction>1</mechanicalReduction>
       </actuator>

Commit message: fixed palm

File: quad_description/urdf/kit_c.urdf (robot description, URDF)
Before this commit: robot quad, 12 links, 11 joints
Joints:
- joint palm_riser: limit lower=0 upper=0.1 effort=2.5 velocity=1.0 -> (none); type prismatic -> fixed

File: quad_description/urdf/my_gripper.xacro (robot description, xacro)
@@ -159,7 +159,6 @@
       <child link="right_finger_tip"/>
     </joint>
-    <joint name="palm_riser" type="prismatic">
-      <axis xyz="0 0 1"/>
-      <limit lower="0" upper="0.1" effort="2.5" velocity="1.0"/>
+    <joint name="palm_riser" type="fixed">
+      <axis xyz="0 0 1"/>
       <origin rpy="0 0 0" xyz="0 0 0"/>
       <parent link="riser"/>
@@ -207,5 +206,5 @@
       </actuator>
     </transmission>
-    <transmission name="tran5">
+    <!--<transmission name="tran5">
       <type>transmission_interface/SimpleTransmission</type>
       <joint name="palm_riser">
@@ -216,5 +215,5 @@
         <mechanicalReduction>1</mechanicalReduction>
       </actuator>
-    </transmission>
+    </transmission>-->
   <gazebo>
     <plugin name="gazebo_ros_control" filename="libgazebo_ros_control.so">

Commit message: only quadrotor

File: quad_description/urdf/kit_c.urdf (robot description, URDF)
Before this commit: robot quad, 12 links, 11 joints
Links:
- removed link left_finger
- removed link left_finger_tip
- removed link palm
- removed link right_finger
- removed link right_finger_tip
- removed link riser
Joints:
- removed joint base1_joint
- removed joint left_finger_tip
- removed joint palm_left_finger
- removed joint palm_right_finger
- removed joint palm_riser
- removed joint right_finger_tip

File: quad_description/urdf/kit_c.xacro (robot description, xacro)
@@ -133,5 +133,3 @@
     <xacro:insert_block name="rotor_inertia" />
   </xacro:vertical_rotor>
-  <xacro:include filename="$(find quad_description)/urdf/my_gripper.xacro"/>
-  <my_gripper_macro/>
 </robot>
