Commit message: Update my_gripper.xacro

File: quad_description/urdf/my_gripper.xacro (robot description, xacro)
@@ -32,6 +32,6 @@
       </collision>
       <inertial>
-        <mass value="0.2"/>
-        <inertia ixx="0.01" ixy="0.0" ixz="0.0" iyy="0.01" iyz="0.0" izz="0.01"/>
+        <mass value="0.02"/>
+        <inertia ixx="0.0000125" ixy="0.0" ixz="0.0" iyy="0.0000125" iyz="0.0" izz="0.0000125"/>
       </inertial>
     </link>
@@ -51,6 +51,6 @@
       </collision>
       <inertial>
-        <mass value="0.1"/>
-        <inertia ixx="0.01" ixy="0.0" ixz="0.0" iyy="0.01" iyz="0.0" izz="0.01"/>
+        <mass value="0.01"/>
+        <inertia ixx="0.0000125" ixy="0.0" ixz="0.0" iyy="0.0000125" iyz="0.0" izz="0.0000125"/>
       </inertial>
     </link>
@@ -70,6 +70,6 @@
       </collision>
       <inertial>
-        <mass value="0.1"/>
-        <inertia ixx="0.01" ixy="0.0" ixz="0.0" iyy="0.01" iyz="0.0" izz="0.01"/>
+        <mass value="0.01"/>
+        <inertia ixx="0.0000125" ixy="0.0" ixz="0.0" iyy="0.0000125" iyz="0.0" izz="0.0000125"/>
       </inertial>
     </link>
@@ -89,6 +89,6 @@
       </collision>
       <inertial>
-        <mass value="0.1"/>
-        <inertia ixx="0.01" ixy="0.0" ixz="0.0" iyy="0.01" iyz="0.0" izz="0.01"/>
+        <mass value="0.01"/>
+        <inertia ixx="0.0000125" ixy="0.0" ixz="0.0" iyy="0.0000125" iyz="0.0" izz="0.0000125"/>
       </inertial>
     </link>
@@ -108,6 +108,6 @@
       </collision>
       <inertial>
-        <mass value="0.1"/>
-        <inertia ixx="0.01" ixy="0.0" ixz="0.0" iyy="0.01" iyz="0.0" izz="0.01"/>
+        <mass value="0.01"/>
+        <inertia ixx="0.0000125" ixy="0.0" ixz="0.0" iyy="0.0000125" iyz="0.0" izz="0.0000125"/>
       </inertial>
     </link>
@@ -127,6 +127,6 @@
       </collision>
       <inertial>
-        <mass value="0.1"/>
-        <inertia ixx="0.01" ixy="0.0" ixz="0.0" iyy="0.01" iyz="0.0" izz="0.01"/>
+        <mass value="0.01"/>
+        <inertia ixx="0.0000125" ixy="0.0" ixz="0.0" iyy="0.0000125" iyz="0.0" izz="0.0000125"/>
       </inertial>
     </link>
